File: FirstPCB/FirstPCB.sch (KiCad schematic (older format))
At the start: 8 parts

Commit message: rough PCB design done
Parts:
- C1, C2: renamed from C?; value C -> 100n; footprint (none) -> Capacitor_THT:C_Radial_D5.0mm_H5.0mm_P2.00mm
- J1, J2: renamed from J?; footprint (none) -> Connector_PinHeader_2.54mm:PinHeader_1x02_P2.54mm_Vertical
- J3: renamed from J?; footprint (none) -> Connector_PinHeader_2.54mm:PinHeader_1x03_P2.54mm_Vertical
- R1, R2: renamed from R?; value R -> 10k; footprint (none) -> Resistor_THT:R_Axial_DIN0207_L6.3mm_D2.5mm_P7.62mm_Horizontal
- U1: renamed from U?; footprint (none) -> FirstPCB:AD711_PDIP; Digikey (none) -> AD711JNZ-ND
Other:
- moved on the sheet: C1, C2, J1, J2, J3, R1, R2, U1
